Commit message: Model for fully_actuated with tilted rotors

File: models/mrs_robots_description/urdf/fully_actuated.xacro (robot description, xacro)
@@ -280,5 +280,5 @@
     parent="base_link"
     color="Black">
-    <origin xyz="${arm_length * cos30} -${arm_length * sin30} ${arm_height - body_height/2}" rpy="0 0 0" />
+    <origin xyz="${arm_length * cos30} -${arm_length * sin30} ${arm_height - body_height/2}" rpy="0 -0.52 0" />
   </xacro:visual_macro>
   <xacro:visual_macro
@@ -289,5 +289,5 @@
     parent="base_link"
     color="Black">
-    <origin xyz="0 -${arm_length} ${arm_height - body_height/2}" rpy="0 0 0" />
+    <origin xyz="0 -${arm_length} ${arm_height - body_height/2}" rpy="0.0 0.52 1.04" />
   </xacro:visual_macro>
   <xacro:visual_macro
@@ -298,5 +298,5 @@
     parent="base_link"
     color="Black">
-    <origin xyz="-${arm_length * cos30} -${arm_length * sin30} ${arm_height - body_height/2}" rpy="0 0 0" />
+    <origin xyz="-${arm_length * cos30} -${arm_length * sin30} ${arm_height - body_height/2}" rpy="0 0.52 -1.04" />
   </xacro:visual_macro>
   <xacro:visual_macro
@@ -307,5 +307,5 @@
     parent="base_link"
     color="Black">
-    <origin xyz="${arm_length * cos30} ${arm_length * sin30} ${arm_height - body_height/2}" rpy="0 0 0" />
+    <origin xyz="${arm_length * cos30} ${arm_length * sin30} ${arm_height - body_height/2}" rpy="0 -0.52 2.09439510239" />
   </xacro:visual_macro>
   <xacro:visual_macro
@@ -316,5 +316,5 @@
     parent="base_link"
     color="Black">
-    <origin xyz="0 ${arm_length} ${arm_height - body_height/2}" rpy="0 0 0" />
+    <origin xyz="0 ${arm_length} ${arm_height - body_height/2}" rpy="0 -0.52 -2.09439510239" />
   </xacro:visual_macro>
   <xacro:visual_macro
@@ -325,5 +325,5 @@
     parent="base_link"
     color="Black">
-    <origin xyz="-${arm_length * cos30} ${arm_length * sin30} ${arm_height - body_height/2}" rpy="0 0 0" />
+    <origin xyz="-${arm_length * cos30} ${arm_length * sin30} ${arm_height - body_height/2}" rpy="0 0.52 -3.1415" />
   </xacro:visual_macro>
   <!--}-->
@@ -347,5 +347,5 @@
     mesh_scale="${mesh_scale_prop_cw}"
     color="White">
-    <origin xyz="0 -${arm_length} ${arm_height + rotor_offset_top - body_height/2}" rpy="0 0 0" />
+    <origin xyz="0 -${arm_length} ${arm_height + rotor_offset_top - body_height/2}" rpy="0.0 0.52 1.04" />
     <xacro:insert_block name="rotor_inertia" />
   </xacro:vertical_rotor>
@@ -368,5 +368,5 @@
     mesh_scale="${mesh_scale_prop_ccw}"
     color="White">
-    <origin xyz="0 ${arm_length} ${arm_height + rotor_offset_top - body_height/2}" rpy="0 0 0" />
+    <origin xyz="0 ${arm_length} ${arm_height + rotor_offset_top - body_height/2}" rpy="0 -0.52 -2.09439510239" />
     <xacro:insert_block name="rotor_inertia" />
   </xacro:vertical_rotor>
@@ -389,5 +389,5 @@
     mesh_scale="${mesh_scale_prop_cw}"
     color="White">
-    <origin xyz="${arm_length * cos30} ${arm_length * sin30} ${arm_height + rotor_offset_top - body_height/2}" rpy="0 0 0" />
+    <origin xyz="${arm_length * cos30} ${arm_length * sin30} ${arm_height + rotor_offset_top - body_height/2}" rpy="0 -0.52 2.09439510239" />
     <xacro:insert_block name="rotor_inertia" />
   </xacro:vertical_rotor>
@@ -410,5 +410,5 @@
     mesh_scale="${mesh_scale_prop_ccw}"
     color="White">
-    <origin xyz="-${arm_length * cos30} -${arm_length * sin30} ${arm_height + rotor_offset_top - body_height/2}" rpy="0 0 0" />
+    <origin xyz="-${arm_length * cos30} -${arm_length * sin30} ${arm_height + rotor_offset_top - body_height/2}" rpy="0 0.52 -1.04" />
     <xacro:insert_block name="rotor_inertia" />
   </xacro:vertical_rotor>
@@ -428,7 +428,7 @@
     rolling_moment_coefficient="${rolling_moment_coefficient}"
     mesh_file="${prop_mesh_file}"
-    mesh_scale="${mesh_scale_prop_cw}"
+    mesh_scale="${mesh_scale_prop_ccw}"
     color="White">
-    <origin xyz="${arm_length * cos30} -${arm_length * sin30} ${arm_height + rotor_offset_top - body_height/2}" rpy="0 0 0" />
+    <origin xyz="${arm_length * cos30} -${arm_length * sin30} ${arm_height + rotor_offset_top - body_height/2}" rpy="0 -0.52 0" />
     <xacro:insert_block name="rotor_inertia" />
   </xacro:vertical_rotor>
@@ -450,5 +450,5 @@
     mesh_scale="${mesh_scale_prop_cw}"
     color="White">
-    <origin xyz="-${arm_length * cos30} ${arm_length * sin30} ${arm_height + rotor_offset_top - body_height/2}" rpy="0 0 0" />
+    <origin xyz="-${arm_length * cos30} ${arm_length * sin30} ${arm_height + rotor_offset_top - body_height/2}" rpy="0 0.52 -3.1415" />
     <xacro:insert_block name="rotor_inertia" />
   </xacro:vertical_rotor>

Commit message: Fixed 3d model fully actuated

File: models/mrs_robots_description/urdf/fully_actuated.xacro (robot description, xacro)
@@ -280,5 +280,5 @@
     parent="base_link"
     color="Black">
-    <origin xyz="${arm_length * cos30} -${arm_length * sin30} ${arm_height - body_height/2}" rpy="0 -0.52 0" />
+    <origin xyz="${arm_length * cos30} -${arm_length * sin30} ${arm_height - body_height/2}" rpy="0.0 -0.52 1.04" />
   </xacro:visual_macro>
   <xacro:visual_macro
@@ -289,5 +289,5 @@
     parent="base_link"
     color="Black">
-    <origin xyz="0 -${arm_length} ${arm_height - body_height/2}" rpy="0.0 0.52 1.04" />
+    <origin xyz="0 -${arm_length} ${arm_height - body_height/2}" rpy="0 0.52 0" />
   </xacro:visual_macro>
   <xacro:visual_macro
@@ -298,5 +298,5 @@
     parent="base_link"
     color="Black">
-    <origin xyz="-${arm_length * cos30} -${arm_length * sin30} ${arm_height - body_height/2}" rpy="0 0.52 -1.04" />
+    <origin xyz="-${arm_length * cos30} -${arm_length * sin30} ${arm_height - body_height/2}" rpy="0 -0.52 -1.04" />
   </xacro:visual_macro>
   <xacro:visual_macro
@@ -307,5 +307,5 @@
     parent="base_link"
     color="Black">
-    <origin xyz="${arm_length * cos30} ${arm_length * sin30} ${arm_height - body_height/2}" rpy="0 -0.52 2.09439510239" />
+    <origin xyz="${arm_length * cos30} ${arm_length * sin30} ${arm_height - body_height/2}" rpy="0 0.52 2.09439510239" />
   </xacro:visual_macro>
   <xacro:visual_macro
@@ -316,5 +316,5 @@
     parent="base_link"
     color="Black">
-    <origin xyz="0 ${arm_length} ${arm_height - body_height/2}" rpy="0 -0.52 -2.09439510239" />
+    <origin xyz="0 ${arm_length} ${arm_height - body_height/2}" rpy="0 -0.52 -3.1415" />
   </xacro:visual_macro>
   <xacro:visual_macro
@@ -325,5 +325,5 @@
     parent="base_link"
     color="Black">
-    <origin xyz="-${arm_length * cos30} ${arm_length * sin30} ${arm_height - body_height/2}" rpy="0 0.52 -3.1415" />
+    <origin xyz="-${arm_length * cos30} ${arm_length * sin30} ${arm_height - body_height/2}" rpy="0 0.52 -2.09439510239" />
   </xacro:visual_macro>
   <!--}-->
@@ -347,5 +347,5 @@
     mesh_scale="${mesh_scale_prop_cw}"
     color="White">
-    <origin xyz="0 -${arm_length} ${arm_height + rotor_offset_top - body_height/2}" rpy="0.0 0.52 1.04" />
+    <origin xyz="0 -${arm_length} ${arm_height + rotor_offset_top - body_height/2}" rpy="0 0.52 0" />
     <xacro:insert_block name="rotor_inertia" />
   </xacro:vertical_rotor>
@@ -368,5 +368,5 @@
     mesh_scale="${mesh_scale_prop_ccw}"
     color="White">
-    <origin xyz="0 ${arm_length} ${arm_height + rotor_offset_top - body_height/2}" rpy="0 -0.52 -2.09439510239" />
+    <origin xyz="0 ${arm_length} ${arm_height + rotor_offset_top - body_height/2}" rpy="0 -0.52 -3.1415" />
     <xacro:insert_block name="rotor_inertia" />
   </xacro:vertical_rotor>
@@ -389,5 +389,5 @@
     mesh_scale="${mesh_scale_prop_cw}"
     color="White">
-    <origin xyz="${arm_length * cos30} ${arm_length * sin30} ${arm_height + rotor_offset_top - body_height/2}" rpy="0 -0.52 2.09439510239" />
+    <origin xyz="${arm_length * cos30} ${arm_length * sin30} ${arm_height + rotor_offset_top - body_height/2}" rpy="0 0.52 2.09439510239" />
     <xacro:insert_block name="rotor_inertia" />
   </xacro:vertical_rotor>
@@ -410,5 +410,5 @@
     mesh_scale="${mesh_scale_prop_ccw}"
     color="White">
-    <origin xyz="-${arm_length * cos30} -${arm_length * sin30} ${arm_height + rotor_offset_top - body_height/2}" rpy="0 0.52 -1.04" />
+    <origin xyz="-${arm_length * cos30} -${arm_length * sin30} ${arm_height + rotor_offset_top - body_height/2}" rpy="0 -0.52 -1.04" />
     <xacro:insert_block name="rotor_inertia" />
   </xacro:vertical_rotor>
@@ -430,5 +430,5 @@
     mesh_scale="${mesh_scale_prop_ccw}"
     color="White">
-    <origin xyz="${arm_length * cos30} -${arm_length * sin30} ${arm_height + rotor_offset_top - body_height/2}" rpy="0 -0.52 0" />
+    <origin xyz="${arm_length * cos30} -${arm_length * sin30} ${arm_height + rotor_offset_top - body_height/2}" rpy="0.0 -0.52 1.04" />
     <xacro:insert_block name="rotor_inertia" />
   </xacro:vertical_rotor>
@@ -450,5 +450,5 @@
     mesh_scale="${mesh_scale_prop_cw}"
     color="White">
-    <origin xyz="-${arm_length * cos30} ${arm_length * sin30} ${arm_height + rotor_offset_top - body_height/2}" rpy="0 0.52 -3.1415" />
+    <origin xyz="-${arm_length * cos30} ${arm_length * sin30} ${arm_height + rotor_offset_top - body_height/2}" rpy="0 0.52 -2.09439510239" />
     <xacro:insert_block name="rotor_inertia" />
   </xacro:vertical_rotor>
